File: Earring - Cat 2.0.kicad_pcb (KiCad board)
At the start: 2 copper layers, 26 x 28.5 mm, 17 parts, among them Q1 2N3904U, Q2 2N3904U, SW1 SW_SPST

Commit message: boards fabricated
Parts:
- added R6: 0R (jumper), Resistor_SMD:R_0805_2012Metric, F.Cu at (29.9, 35.0)
- moved Q2 2.83 mm to (23.5, 36.4), turned to 0 degrees
- moved Q1 2.40 mm to (37.1, 36.4), turned to 0 degrees
- moved G*** 1.02 mm to (23.2, 22.0)
- moved R1 1.00 mm to (23.0, 27.0)
- moved R2 1.00 mm to (25.5, 27.0)
- moved R3 1.00 mm to (34.5, 27.0)
- moved R4 1.00 mm to (37.0, 27.0)
- moved G*** 0.61 mm to (36.6, 21.6)
- moved D1 0.50 mm to (24.0, 30.0)
- moved D2 0.50 mm to (36.0, 30.0)
- moved C1 0.34 mm to (27.4, 32.8)
- moved C2 0.32 mm to (32.6, 32.8)
- moved SW1 0.30 mm to (30.0, 41.8)
- moved H1 0.10 mm to (30.0, 20.6)
Connections:
- C1 pad 2: Net-(Q1-B) -> Net-(C1-Pad2)
- Q1 pad 1: GND -> Net-(Q1-B)
- Q1 pad 2: Net-(Q1-B) -> Net-(D2-K)
- Q1 pad 3: Net-(D2-K) -> GND
- Q2 pad 1: GND -> Net-(Q2-B)
- Q2 pad 2: Net-(Q2-B) -> Net-(D1-K)
- Q2 pad 3: Net-(D1-K) -> GND
- R2 pad 2: Net-(Q1-B) -> Net-(C1-Pad2)
Routing:
- net GND: track 0.00 -> 52.4 mm, vias 10 -> 2
- net Net-(BT1-+): track 13.0 -> 41.8 mm
- net Net-(Q1-B): track 26.7 -> 4.38 mm, vias 2 -> 0
- net Net-(C1-Pad2): track 0.00 -> 8.53 mm
- net Net-(D1-K): track 5.80 -> 13.7 mm
- net Net-(Q2-B): track 25.2 -> 19.0 mm
- net Net-(SW1-B): track 39.2 -> 34.4 mm, vias 1 -> 0
- net Net-(D2-K): track 8.54 -> 10.3 mm
- net Net-(D2-A): track 2.75 -> 2.25 mm
- net Net-(D1-A): track 2.75 -> 2.25 mm
- added copper zone on B.Cu, net (none)
- added copper zone on F.Cu, net (none)
- removed copper zone on B.Cu, net GND
- removed copper zone on F.Cu, net GND
