File: Earring - Cat 2.0.kicad_sch (KiCad schematic)
At the start: 13 parts, among them Q1 2N3904U, Q2 2N3904U, SW1 SW_SPST

Commit message: updated readme
Parts:
- added R6: 0R (jumper), Resistor_SMD:R_0805_2012Metric, symbol Device:R_Small
Connections:
- net at C1.2, R2.2: now also R6.1; no longer Q1.1 (B)
- new net: Q1.1 (B), R6.2
Changed lines of the file:
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@@
 	(wire
 		(pts
-			(xy 124.46 81.28) (xy 116.84 81.28)
+			(xy 124.46 81.28) (xy 123.19 81.28)
 		)
 		(stroke
@@
 		(pts
 			(xy 85.09 38.1) (xy 91.44 38.1)
+		)
+		(stroke
+			(width 0)
+			(type default)
+		)
+	)
+	(wire
+		(pts
+			(xy 118.11 81.28) (xy 116.84 81.28)
 		)
 		(stroke
@@
 					(unit 1)
 				)
+			)
+		)
+	)
+	(symbol
+		(lib_id "Device:R_Small")
+		(at 120.65 81.28 90)
+		(unit 1)
+		(exclude_from_sim no)
+		(in_bom yes)
+		(on_board yes)
+		(dnp no)
+		(fields_autoplaced yes)
+		(property "Reference" "R6"
+			(at 120.65 76.2 90)
+			(effects
+				(font
+					(size 1.27 1.27)
+				)
+			)
+		)
+		(property "Value" "0R (jumper)"
+			(at 120.65 78.74 90)
+			(effects
+				(font
+					(size 1.27 1.27)
+				)
+			)
+		)
+		(property "Footprint" "Resistor_SMD:R_0805_2012Metric"
+			(at 120.65 81.28 0)
+			(effects
+				(font
+					(size 1.27 1.27)
+				)
+				(hide yes)
+			)
+		)
+		(property "Datasheet" "~"
+			(at 120.65 81.28 0)
+			(effects
+				(font
+					(size 1.27 1.27)
+				)
+				(hide yes)
+			)
+		)
+		(property "Description" "Resistor, small symbol"
+			(at 120.65 81.28 0)
+			(effects
+				(font
+					(size 1.27 1.27)
+				)
+				(hide yes)
+			)
+		)
+		(pin "1"
+		)
+		(pin "2"
+		)
+		(instances
+			(project ""
+				(path "/ff3e0cf6-72c2-4d8a-868c-e0988eb4f32e"
+					(reference "R6")
+					(unit 1)
+				)
