File: Earring - Cat 2.0.kicad_sch (KiCad schematic)
At the start: 11 parts, among them Q1 2N3904U, Q2 2N3904U

Commit message: render
Parts:
- added H1: MountingHole, MountingHole:MountingHole_2.2mm_M2_DIN965_Pad, symbol Mechanical:MountingHole
- added SW1: SW_SPST, Soso:DIP switch 1P THT, symbol Switch:SW_SPST
Connections:
- net at R1.1, R2.1, R3.1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: now also SW1.2 (B); no longer BT1.1 (+)
- new net: BT1.1 (+), SW1.1 (A)
Changed lines of the file:
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@@
 	(wire
 		(pts
-			(xy 71.12 38.1) (xy 91.44 38.1)
+			(xy 71.12 38.1) (xy 74.93 38.1)
 		)
 		(stroke
@@
 		(pts
 			(xy 105.41 50.8) (xy 105.41 72.39)
+		)
+		(stroke
+			(width 0)
+			(type default)
+		)
+	)
+	(wire
+		(pts
+			(xy 85.09 38.1) (xy 91.44 38.1)
 		)
 		(stroke
@@
 					(unit 1)
 				)
+			)
+		)
+	)
+	(symbol
+		(lib_id "Switch:SW_SPST")
+		(at 80.01 38.1 0)
+		(unit 1)
+		(exclude_from_sim no)
+		(in_bom yes)
+		(on_board yes)
+		(dnp no)
+		(property "Reference" "SW1"
+			(at 80.264 42.672 90)
+			(effects
+				(font
+					(size 1.27 1.27)
+				)
+				(justify right)
+			)
+		)
+		(property "Value" "SW_SPST"
+			(at 77.724 40.386 90)
+			(effects
+				(font
+					(size 1.27 1.27)
+				)
+				(justify right)
+			)
+		)
+		(property "Footprint" "Soso:DIP switch 1P THT"
+			(at 80.01 38.1 0)
+			(effects
+				(font
+					(size 1.27 1.27)
+				)
+				(hide yes)
+			)
+		)
+		(property "Datasheet" "~"
+			(at 80.01 38.1 0)
+			(effects
+				(font
+					(size 1.27 1.27)
+				)
+				(hide yes)
+			)
+		)
+		(property "Description" "Single Pole Single Throw (SPST) switch"
+			(at 80.01 38.1 0)
+			(effects
+				(font
+					(size 1.27 1.27)
+				)
+				(hide yes)
+			)
+		)
+		(pin "2"
+		)
+		(pin "1"
+		)
+		(instances
+			(project "Earring - Cat 2.0"
+				(path "/ff3e0cf6-72c2-4d8a-868c-e0988eb4f32e"
+					(reference "SW1")
+					(unit 1)
+				)
+			)
+		)
+	)
+	(symbol
+		(lib_id "Mechanical:MountingHole")
+		(at 152.4 38.1 0)
+		(unit 1)
+		(exclude_from_sim yes)
+		(in_bom no)
+		(on_board yes)
+		(dnp no)
+		(fields_autoplaced yes)
+		(property "Reference" "H1"
+			(at 154.94 36.8299 0)
+			(effects
+				(font
+					(size 1.27 1.27)
+				)
+				(justify left)
+			)
+		)
+		(property "Value" "MountingHole"
+			(at 154.94 39.3699 0)
+			(effects
+				(font
+					(size 1.27 1.27)
+				)
+				(justify left)
+			)
+		)
+		(property "Footprint" "MountingHole:MountingHole_2.2mm_M2_DIN965_Pad"
+			(at 152.4 38.1 0)
+			(effects
+				(font
+					(size 1.27 1.27)
+				)
+				(hide yes)
+			)
+		)
+		(property "Datasheet" "~"
+			(at 152.4 38.1 0)
+			(effects
+				(font
+					(size 1.27 1.27)
+				)
+				(hide yes)
+			)
+		)
+		(property "Description" "Mounting Hole without connection"
+			(at 152.4 38.1 0)
+			(effects
+				(font
+					(size 1.27 1.27)
+				)
+				(hide yes)
+			)
+		)
+		(instances
+			(project ""
+				(path "/ff3e0cf6-72c2-4d8a-868c-e0988eb4f32e"
+					(reference "H1")
+					(unit 1)
+				)

Commit message: updated prod and media
Parts:
- added R6: 0R (jumper), Resistor_SMD:R_0805_2012Metric, symbol Device:R_Small
Connections:
- net GND: now also Q1.3 (E), Q2.3 (E); no longer Q1.1 (E), Q2.1 (E)
- net at C2.1, D2.1 (K): now also Q1.2 (C); no longer Q1.3 (C)
- net at C1.2, R2.2: now also R6.1; no longer Q1.2 (B)
- net at C2.2, R3.2: now also Q2.1 (B); no longer Q2.2 (B)
- net at C1.1, D1.1 (K): now also Q2.2 (C); no longer Q2.3 (C)
- new net: Q1.1 (B), R6.2
Changed lines of the file:
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@@
 	(wire
 		(pts
-			(xy 124.46 81.28) (xy 116.84 81.28)
+			(xy 124.46 81.28) (xy 123.19 81.28)
 		)
 		(stroke
@@
 		(pts
 			(xy 85.09 38.1) (xy 91.44 38.1)
+		)
+		(stroke
+			(width 0)
+			(type default)
+		)
+	)
+	(wire
+		(pts
+			(xy 118.11 81.28) (xy 116.84 81.28)
 		)
 		(stroke
@@
 	)
 	(symbol
+		(lib_id "Device:R_Small")
+		(at 120.65 81.28 90)
+		(unit 1)
+		(exclude_from_sim no)
+		(in_bom yes)
+		(on_board yes)
+		(dnp no)
+		(fields_autoplaced yes)
+		(property "Reference" "R6"
+			(at 120.65 76.2 90)
+			(effects
+				(font
+					(size 1.27 1.27)
+				)
+			)
+		)
+		(property "Value" "0R (jumper)"
+			(at 120.65 78.74 90)
+			(effects
+				(font
+					(size 1.27 1.27)
+				)
+			)
+		)
+		(property "Footprint" "Resistor_SMD:R_0805_2012Metric"
+			(at 120.65 81.28 0)
+			(effects
+				(font
+					(size 1.27 1.27)
+				)
+				(hide yes)
+			)
+		)
+		(property "Datasheet" "~"
+			(at 120.65 81.28 0)
+			(effects
+				(font
+					(size 1.27 1.27)
+				)
+				(hide yes)
+			)
+		)
+		(property "Description" "Resistor, small symbol"
+			(at 120.65 81.28 0)
+			(effects
+				(font
+					(size 1.27 1.27)
+				)
+				(hide yes)
+			)
+		)
+		(pin "1"
+		)
+		(pin "2"
+		)
+		(instances
+			(project ""
+				(path "/ff3e0cf6-72c2-4d8a-868c-e0988eb4f32e"
+					(reference "R6")
+					(unit 1)
+				)
+			)
+		)
+	)
+	(symbol
 		(lib_id "Device:R")
 		(at 132.08 46.99 0)
@@
 	)
 	(symbol
+		(lib_name "2N3904_1")
 		(lib_id "Transistor_BJT:2N3904")
 		(at 93.98 81.28 0)
@@
 		)
 		(property "Footprint" "Package_TO_SOT_SMD:SOT-89-3"
-			(at 88.9 83.185 0)
+			(at 89.662 89.281 0)
 			(effects
 				(font
@@
 		)
 		(property "Datasheet" "https://www.onsemi.com/pub/Collateral/2N3903-D.PDF"
-			(at 93.98 81.28 0)
+			(at 94.742 87.376 0)
 			(effects
 				(font
@@
 		)
 		(property "Description" "0.2A Ic, 40V Vce, Small Signal NPN Transistor, TO-92"
-			(at 93.98 81.28 0)
+			(at 94.742 88.392 0)
 			(effects
 				(font
@@
 		)
 		(property "Footprint" "Package_TO_SOT_SMD:SOT-89-3"
-			(at 134.62 83.185 0)
+			(at 133.604 89.789 0)
 			(effects
 				(font
@@
 		)
 		(property "Datasheet" "https://www.onsemi.com/pub/Collateral/2N3903-D.PDF"
-			(at 129.54 81.28 0)
+			(at 128.524 87.884 0)
 			(effects
 				(font
@@
 		)
 		(property "Description" "0.2A Ic, 40V Vce, Small Signal NPN Transistor, TO-92"
-			(at 129.54 81.28 0)
-			(effects
-				(font
+			(at 130.302 88.138 0)
+			(effects
+				(font
